File: mcp1640_5v_supply.sch (KiCad schematic (older format))
At the start: 8 parts, among them J1 Conn_01x03, U1 MCP1640CH

Commit message: Another revision
Connections:
- net FBACK: now reaches R2.2, R3.1, U1.4 (VFB)
Changed lines of the file:
@@
 EESchema Schematic File Version 4
-EELAYER 29 0
+EELAYER 30 0
 EELAYER END
 $Descr A4 11693 8268
@@
 Text GLabel 6100 3050 2    50   Input ~ 0
 +5V
+Text GLabel 5400 3350 1    50   Input ~ 0
+FBACK
 $EndSCHEMATC
